File: Nodo/PCB_placa_adaptadora/Mini-Lora.brd (EAGLE design)
At the start: 56.5 x 25.7 mm, 7 parts, among them P1 GND, P2 3v3

Commit message: Corrección el el board de la placa del nodo
Bug detectado por @giltesa
Routing:
- net 3V3: track 68.4 -> 66.8 mm
Changed lines of the file:
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@@
 <wire x1="31.75" y1="24.13" x2="32.131" y2="24.003" width="0.4064" layer="16"/>
 <wire x1="29.21" y1="22.86" x2="28.575" y2="22.225" width="0.4064" layer="16"/>
-<wire x1="66.04" y1="15.24" x2="55.88" y2="5.08" width="0.4064" layer="16"/>
-<wire x1="66.04" y1="24.13" x2="66.04" y2="15.24" width="0.4064" layer="16"/>
-<wire x1="33.02" y1="24.13" x2="66.04" y2="24.13" width="0.4064" layer="16"/>
+<wire x1="65.0494" y1="15.2908" x2="55.88" y2="5.08" width="0.4064" layer="16"/>
+<wire x1="65.0494" y1="24.1808" x2="65.0494" y2="15.2908" width="0.4064" layer="16"/>
+<wire x1="33.02" y1="24.13" x2="65.0494" y2="24.1808" width="0.4064" layer="16"/>
 <wire x1="33.02" y1="24.13" x2="32.131" y2="24.003" width="0.4064" layer="16"/>
 </signal>
